File: electronica/PBC-2/PBC-2.sch (EAGLE design)
At the start: 9 parts

Commit message: fin pcb-2
fin pcb-2
Parts:
- added BTN: 22-23-2021, con-molex:22-23-2021
- added R1: (no value), rcl:R-US_0204/5
Connections:
- new net N$1: BTN-1.S, MEGA.23, R1.1
- net +5V: now also BTN-2.S, MEGA.+5V..
- net GND: now also R1.2
Changed lines of the file:
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@@
 <part name="P+10" library="supply1" deviceset="+5V" device=""/>
 <part name="GND9" library="supply1" deviceset="GND" device=""/>
+<part name="BTN" library="con-molex" deviceset="22-23-2021" device="" value=""/>
+<part name="R1" library="rcl" deviceset="R-US_" device="0204/5"/>
 </parts>
 <sheets>
@@
 <instance part="P+10" gate="1" x="-12.7" y="149.86" rot="MR90"/>
 <instance part="GND9" gate="1" x="-20.32" y="160.02" rot="R180"/>
+<instance part="BTN" gate="-1" x="-45.72" y="93.98" rot="R180"/>
+<instance part="BTN" gate="-2" x="-45.72" y="96.52" rot="R180"/>
+<instance part="R1" gate="G$1" x="-10.16" y="93.98" rot="R90"/>
 </instances>
 <busses>
@@
 <wire x1="-30.48" y1="101.6" x2="-17.78" y2="101.6" width="0.1524" layer="91"/>
 <wire x1="-17.78" y1="101.6" x2="-17.78" y2="99.06" width="0.1524" layer="91"/>
+<pinref part="R1" gate="G$1" pin="2"/>
+<wire x1="-10.16" y1="99.06" x2="-10.16" y2="101.6" width="0.1524" layer="91"/>
+<wire x1="-10.16" y1="101.6" x2="-17.78" y2="101.6" width="0.1524" layer="91"/>
+<junction x="-17.78" y="101.6"/>
 </segment>
 <segment>
@@
 <segment>
 <pinref part="P+5" gate="1" pin="+5V"/>
-<wire x1="-33.02" y1="86.36" x2="-25.4" y2="86.36" width="0.1524" layer="91"/>
+<wire x1="-33.02" y1="86.36" x2="-30.48" y2="86.36" width="0.1524" layer="91"/>
+<pinref part="MEGA" gate="G$1" pin="+5V.."/>
+<wire x1="-30.48" y1="86.36" x2="-22.86" y2="86.36" width="0.1524" layer="91"/>
+<wire x1="-15.24" y1="86.36" x2="-22.86" y2="86.36" width="0.1524" layer="91"/>
+<junction x="-22.86" y="86.36"/>
+<pinref part="BTN" gate="-2" pin="S"/>
+<wire x1="-30.48" y1="86.36" x2="-30.48" y2="96.52" width="0.1524" layer="91"/>
+<wire x1="-30.48" y1="96.52" x2="-43.18" y2="96.52" width="0.1524" layer="91"/>
+<junction x="-30.48" y="86.36"/>
 </segment>
 <segment>
@@
 </segment>
 </net>
+<net name="N$1" class="0">
+<segment>
+<pinref part="BTN" gate="-1" pin="S"/>
+<wire x1="-43.18" y1="93.98" x2="-43.18" y2="83.82" width="0.1524" layer="91"/>
+<wire x1="-43.18" y1="83.82" x2="-22.86" y2="83.82" width="0.1524" layer="91"/>
+<pinref part="MEGA" gate="G$1" pin="23"/>
+<pinref part="R1" gate="G$1" pin="1"/>
+<wire x1="-22.86" y1="83.82" x2="-10.16" y2="83.82" width="0.1524" layer="91"/>
+<wire x1="-10.16" y1="83.82" x2="-10.16" y2="88.9" width="0.1524" layer="91"/>
+<junction x="-22.86" y="83.82"/>
+</segment>
+</net>
