File: electronica/PBC-2/PBC-2.brd (EAGLE design)
At the start: 160 x 100 mm, 9 parts

Commit message: posiciones pcb-2
Parts:
- moved TXT 283.7 mm to (28.7, -76.1)
- moved SV1 200.5 mm to (45.8, 61.0)
- moved PUENTE1 186.0 mm to (76.3, -41.0), turned to 90 degrees
- moved MEGA 170.0 mm to (50.5, -35.0), turned to 180 degrees
- moved PUENTE2 162.1 mm to (-25.0, -41.0), turned to 90 degrees
- moved JP1 160.9 mm to (37.2, -54.4), turned to 270 degrees
- moved VEL 153.2 mm to (-5.25, 46.2)
- moved UNO 140.6 mm to (-34.3, 33.0)
- moved JP2 132.0 mm to (5.95, -76.8), turned to 180 degrees
Connections:
- net ECHO: now also MEGA.48
- net M1ENL: now also MEGA.35
- net M1ENR: now also MEGA.29
- net M1INAL: now also MEGA.31
- net M1INAR: now also MEGA.25
- net M1INBL: now also MEGA.33
- net M1INBR: now also MEGA.27
- net M2ENL: now also MEGA.34
- net M2ENR: now also MEGA.28
- net M2INAL: now also MEGA.30
- net M2INAR: now also MEGA.24
- net M2INBL: now also MEGA.32
- net M2INBR: now also MEGA.26
- net PIXY1: now also MEGA.51
- net PIXY2: now also MEGA.50
- net PIXY3: now also MEGA.53
- net PIXY4: now also MEGA.52
- net TRIG: now also MEGA.49
Other:
- board size 160 x 100 mm -> 210 x 196.1 mm

Commit message: fin pcb-2
fin pcb-2
Parts:
- added BTN: (no value), con-garry:332-02
- added R1: (no value), eagle-ltspice:0204/7
- moved JP2 137.3 mm to (32.0, 58.0), flipped to the bottom, turned to 270 degrees
- moved SV1 80.8 mm to (-34.9, 56.6), flipped to the bottom
- moved VEL 46.2 mm to (1.50, 0.51)
- moved JP1 19.0 mm to (56.0, -51.8), turned to 90 degrees
- moved TXT 5.63 mm to (24.8, -80.1)
- moved UNO 5.41 mm to (-39.7, 33.3)
Connections:
- new net S$1: BTN.2, MEGA.12
- new net S$2: BTN.1, MEGA.13, R1.2
- new net S$3: MEGA.GND, R1.1
- net +5V: now also MEGA.5V..
- net RX-XBEE: no longer JP2.4
Routing:
- net +5V: track 0.00 -> 571.3 mm
- net M1INAL: track 0.00 -> 494.9 mm
- net M1INBL: track 0.00 -> 484.8 mm
- net RX-XBEE: track 0.00 -> 378.8 mm
- net M1ENR: track 0.00 -> 348.5 mm
- net TX-XBEE: track 0.00 -> 344.1 mm
- net M2PWMR: track 0.00 -> 332.2 mm
- net M2INAR: track 0.00 -> 318.2 mm
- net M1ENL: track 0.00 -> 199.7 mm, vias 0 -> 2
- net M2INAL: track 0.00 -> 174.6 mm
- net PIXY3: track 0.00 -> 168.7 mm
- net PIXY2: track 0.00 -> 165.6 mm
- net M2ENL: track 0.00 -> 165.0 mm
- net M1PWML: track 0.00 -> 164.5 mm
- net PIXY4: track 0.00 -> 163.3 mm
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- added copper zone on layer 1, net GND
- added copper zone on layer 16, net GND
Other:
- outline, holes or cut-outs redrawn
- board text added: "C:/Users/carlos hugo/Desktop/github/L16/electronica/PBC-2/InteliRobot.bmp"
- board text added: "C:/Users/carlos hugo/Desktop/github/L16/electronica/PBC-2/yoHagoRobots.bmp"
- board text added: "InteliRobot"

Commit message: ELECTRONICA
FIN DE LOS DISEÑOS
Other:
- board text removed: "C:/Users/carlos hugo/Desktop/github/L16/electronica/PBC-2/yoHagoRobots.bmp"

Commit message: ELECTRONICA FIN
diseño final de las pcb's y creacion de gerbers
Routing:
- net M1INBL: track 484.8 -> 483.9 mm
- net TX-XBEE: track 344.1 -> 344.8 mm
Changed lines of the file:
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@@
 <setting verticaltext="up"/>
 </settings>
-<grid distance="1" unitdist="mm" unit="mm" style="lines" multiple="1" display="yes" altdistance="1" altunitdist="mm" altunit="mm"/>
+<grid distance="0.003125" unitdist="mic" unit="mm" style="lines" multiple="1" display="yes" altdistance="0.003125" altunitdist="mic" altunit="mm"/>
 <layers>
 <layer number="1" name="Top" color="4" fill="1" visible="yes" active="yes"/>
@@
 <layer number="27" name="tValues" color="7" fill="1" visible="yes" active="yes"/>
 <layer number="28" name="bValues" color="7" fill="1" visible="yes" active="yes"/>
-<layer number="29" name="tStop" color="7" fill="3" visible="yes" active="yes"/>
-<layer number="30" name="bStop" color="7" fill="6" visible="yes" active="yes"/>
-<layer number="31" name="tCream" color="7" fill="4" visible="yes" active="yes"/>
-<layer number="32" name="bCream" color="7" fill="5" visible="yes" active="yes"/>
-<layer number="33" name="tFinish" color="6" fill="3" visible="yes" active="yes"/>
-<layer number="34" name="bFinish" color="6" fill="6" visible="yes" active="yes"/>
-<layer number="35" name="tGlue" color="7" fill="4" visible="yes" active="yes"/>
-<layer number="36" name="bGlue" color="7" fill="5" visible="yes" active="yes"/>
+<layer number="29" name="tStop" color="7" fill="3" visible="no" active="yes"/>
+<layer number="30" name="bStop" color="7" fill="6" visible="no" active="yes"/>
+<layer number="31" name="tCream" color="7" fill="4" visible="no" active="yes"/>
+<layer number="32" name="bCream" color="7" fill="5" visible="no" active="yes"/>
+<layer number="33" name="tFinish" color="6" fill="3" visible="no" active="yes"/>
+<layer number="34" name="bFinish" color="6" fill="6" visible="no" active="yes"/>
+<layer number="35" name="tGlue" color="7" fill="4" visible="no" active="yes"/>
+<layer number="36" name="bGlue" color="7" fill="5" visible="no" active="yes"/>
 <layer number="37" name="tTest" color="7" fill="1" visible="yes" active="yes"/>
 <layer number="38" name="bTest" color="7" fill="1" visible="yes" active="yes"/>
@@
 <wire x1="4.8128" y1="80.6144" x2="3.9834875" y2="81.4437125" width="1.016" layer="16"/>
 <wire x1="3.9834875" y1="81.4437125" x2="3.9834875" y2="86.06156875" width="1.016" layer="16"/>
-<wire x1="29.4784" y1="87.232" x2="27.593128125" y2="89.117271875" width="1.016" layer="16"/>
-<wire x1="27.593128125" y1="89.117271875" x2="7.039190625" y2="89.117271875" width="1.016" layer="16"/>
-<wire x1="7.039190625" y1="89.117271875" x2="3.9834875" y2="86.06156875" width="1.016" layer="16"/>
+<wire x1="29.4784" y1="87.232" x2="28.65995" y2="88.05045" width="1.016" layer="16"/>
+<wire x1="28.65995" y1="88.05045" x2="5.97236875" y2="88.05045" width="1.016" layer="16"/>
+<wire x1="5.97236875" y1="88.05045" x2="3.9834875" y2="86.06156875" width="1.016" layer="16"/>
 </signal>
 <signal name="M1ENL">
@@
 <wire x1="-36.173421875" y1="56.571940625" x2="-38.458503125" y2="58.857021875" width="1.016" layer="1"/>
 <wire x1="-38.458503125" y1="58.857021875" x2="-38.458503125" y2="78.226715625" width="1.016" layer="1"/>
-<wire x1="-38.458503125" y1="78.226715625" x2="-27.631634375" y2="89.053584375" width="1.016" layer="1"/>
 <wire x1="-5.657653125" y1="84.138325" x2="-5.657653125" y2="86.402403125" width="1.016" layer="1"/>
-<wire x1="-5.657653125" y1="86.402403125" x2="-8.308834375" y2="89.053584375" width="1.016" layer="1"/>
-<wire x1="-8.308834375" y1="89.053584375" x2="-27.631634375" y2="89.053584375" width="1.016" layer="1"/>
+<wire x1="-5.657653125" y1="86.402403125" x2="-7.940528125" y2="88.685278125" width="1.016" layer="1"/>
+<wire x1="-7.940528125" y1="88.685278125" x2="-27.999940625" y2="88.685278125" width="1.016" layer="1"/>
+<wire x1="-27.999940625" y1="88.685278125" x2="-38.458503125" y2="78.226715625" width="1.016" layer="1"/>
 </signal>
 <signal name="MISO">
@@
 <wire x1="-8.4224" y1="67.9808" x2="27.6736" y2="67.9808" width="1" layer="16"/>
 <wire x1="-10.8288" y1="65.5744" x2="-8.4224" y2="67.9808" width="1" layer="16"/>
-<wire x1="-69.184" y1="65.5744" x2="-10.8288" y2="65.5744" width="1" layer="16"/>
-<wire x1="-92.0448" y1="42.7136" x2="-69.184" y2="65.5744" width="1" layer="16"/>
-<wire x1="-92.0448" y1="19.2512" x2="-92.0448" y2="42.7136" width="1" layer="16"/>
+<wire x1="-69.184" y1="65.5744" x2="-68.469071875" y2="65.5744" width="1" layer="16"/>
+<wire x1="-68.469071875" y1="65.5744" x2="-10.8288" y2="65.5744" width="1" layer="16"/>
 <wire x1="-96.8576" y1="14.4384" x2="-92.0448" y2="19.2512" width="1" layer="16"/>
 <wire x1="-96.8576" y1="-25.8688" x2="-96.8576" y2="14.4384" width="1" layer="16"/>
@@
 <wire x1="11.06080625" y1="-88.12189375" x2="12.43" y2="-86.7527" width="1.016" layer="16"/>
 <wire x1="12.43" y1="-86.7527" x2="12.43" y2="-85.8" width="1.016" layer="16"/>
+<wire x1="-92.0448" y1="19.2512" x2="-79.3977875" y2="31.8982125" width="1.016" layer="16"/>
+<wire x1="-79.3977875" y1="31.8982125" x2="-79.3977875" y2="55.35928125" width="1.016" layer="16"/>
+<wire x1="-79.3977875" y1="55.35928125" x2="-69.18266875" y2="65.5744" width="1.016" layer="16"/>
+<wire x1="-69.18266875" y1="65.5744" x2="-68.469071875" y2="65.5744" width="1.016" layer="16"/>
 </signal>
 <signal name="RX-XBEE">
 <contactref element="MEGA" pad="1"/>
-<wire x1="-93.248" y1="19.8528" x2="-93.248" y2="43.3152" width="1" layer="16"/>
 <wire x1="-98.0608" y1="15.04" x2="-93.248" y2="19.8528" width="1" layer="16"/>
 <wire x1="-98.0608" y1="-26.4704" x2="-98.0608" y2="15.04" width="1" layer="16"/>
@@
 <wire x1="35.23620625" y1="63.52623125" x2="35.23620625" y2="70.17206875" width="1.016" layer="16"/>
 <wire x1="35.23620625" y1="70.17206875" x2="30.5110375" y2="74.8972375" width="1.016" layer="16"/>
-<wire x1="-93.248" y1="43.3152" x2="-61.6659625" y2="74.8972375" width="1.016" layer="16"/>
-<wire x1="-61.6659625" y1="74.8972375" x2="30.5110375" y2="74.8972375" width="1.016" layer="16"/>
+<wire x1="-61.90074375" y1="74.8972375" x2="30.5110375" y2="74.8972375" width="1.016" layer="16"/>
+<wire x1="-93.248" y1="19.8528" x2="-81.504528125" y2="31.596271875" width="1.016" layer="16"/>
+<wire x1="-81.504528125" y1="31.596271875" x2="-81.504528125" y2="55.293453125" width="1.016" layer="16"/>
+<wire x1="-81.504528125" y1="55.293453125" x2="-61.90074375" y2="74.8972375" width="1.016" layer="16"/>
 </signal>
 <signal name="S$1">
