File: electronica/PBC-1/PBC-1.sch (EAGLE design)
At the start: 86 parts

Commit message: diagrama pcb2
diagrama de la pcb de arriba y prueba de la comunicacion serial
Parts:
- IR-TRAN, LT-TRAN: device linear:7805TV -> linear:7805T
Connections:
- net +5V-LT: now also LT-MULT-1P.VCC, LT-MULT-2P.VCC
- net GND: no longer LT-MULT-1P.VCC, LT-MULT-2P.VCC
Changed lines of the file:
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@@
 <setting verticaltext="up"/>
 </settings>
-<grid distance="0.1" unitdist="inch" unit="inch" style="lines" multiple="1" display="yes" altdistance="0.01" altunitdist="inch" altunit="inch"/>
+<grid distance="0.1" unitdist="inch" unit="inch" style="lines" multiple="1" display="no" altdistance="0.01" altunitdist="inch" altunit="inch"/>
 <layers>
 <layer number="1" name="Top" color="4" fill="1" visible="no" active="no"/>
@@
 </classes>
 <parts>
-<part name="IR-TRAN" library="linear" deviceset="78*" device="TV" technology="05" value="7805"/>
+<part name="IR-TRAN" library="linear" deviceset="78*" device="T" technology="05" value="7805"/>
 <part name="IR-RC2" library="resistor" deviceset="CPOL-EU" device="TT5D9" value="10uf"/>
 <part name="IR-RC1" library="resistor" deviceset="CPOL-EU" device="TT5D9" value="10uf"/>
@@
 <part name="IRDP" library="tsop" deviceset="TSOP1840" device="" value="TSOP2240"/>
 <part name="GND7" library="supply1" deviceset="GND" device=""/>
-<part name="LT-TRAN" library="linear" deviceset="78*" device="TV" technology="05" value="7805"/>
+<part name="LT-TRAN" library="linear" deviceset="78*" device="T" technology="05" value="7805"/>
 <part name="LT-RC1" library="resistor" deviceset="CPOL-EU" device="TT5D9" value="10uf"/>
 <part name="LT-RC2" library="resistor" deviceset="CPOL-EU" device="TT5D9" value="10uf"/>
@@
 </segment>
 <segment>
+<pinref part="S2P" gate="-5" pin="S"/>
 <pinref part="GND13" gate="1" pin="GND"/>
-<pinref part="S2P" gate="-5" pin="S"/>
-<wire x1="-83.82" y1="127" x2="-83.82" y2="124.46" width="0.1524" layer="91"/>
 <pinref part="S2P" gate="-3" pin="S"/>
 <wire x1="-81.28" y1="124.46" x2="-81.28" y2="127" width="0.1524" layer="91"/>
 <wire x1="-81.28" y1="127" x2="-83.82" y2="127" width="0.1524" layer="91"/>
 <junction x="-83.82" y="127"/>
-<pinref part="LT-MULT-2" gate="P" pin="VCC"/>
-<pinref part="LT-MULT-1" gate="P" pin="VCC"/>
-<wire x1="-88.9" y1="139.7" x2="-88.9" y2="134.62" width="0.1524" layer="91"/>
-<wire x1="-88.9" y1="134.62" x2="-83.82" y2="134.62" width="0.1524" layer="91"/>
-<wire x1="-83.82" y1="134.62" x2="-83.82" y2="127" width="0.1524" layer="91"/>
-<junction x="-88.9" y="134.62"/>
+<wire x1="-83.82" y1="127" x2="-83.82" y2="124.46" width="0.1524" layer="91"/>
 </segment>
 <segment>
@@
 <pinref part="S2P" gate="-1" pin="S"/>
 <wire x1="-78.74" y1="127" x2="-78.74" y2="124.46" width="0.1524" layer="91"/>
-</segment>
-<segment>
+<pinref part="LT-MULT-2" gate="P" pin="VCC"/>
+<pinref part="LT-MULT-1" gate="P" pin="VCC"/>
+<wire x1="-88.9" y1="139.7" x2="-88.9" y2="134.62" width="0.1524" layer="91"/>
+<wire x1="-88.9" y1="134.62" x2="-76.2" y2="134.62" width="0.1524" layer="91"/>
+<wire x1="-76.2" y1="134.62" x2="-76.2" y2="127" width="0.1524" layer="91"/>
+<junction x="-88.9" y="134.62"/>
+<wire x1="-76.2" y1="127" x2="-78.74" y2="127" width="0.1524" layer="91"/>
+<junction x="-78.74" y="127"/>
+</segment>
+<segment>

Commit message: fin pcb-2
fin pcb-2
Parts:
- removed CS-BTN, IR-BTN, LT-BTN: RDT1034, switch:RDT1034
- removed IR-MULT-L, IR-MULT-R, LT-MULT-1, LT-MULT-2: 74LS151N, 74xx-us:74LS151N
- removed LT-AT: ATMEGA328P-PU, Atmel_By_element14_Batch_1-00:ATMEGA328P-PU
- removed LT-ATC1, LT-ATC2: 22 pF, capacitor-wima:C2,5-3
- removed LT-CR: 16 MHz, crystal:CRYSTALHC49U70
- removed LT-LED: (no value), led:LED5MM
- removed LT-R1: 10k, rcl:R-US_0204/7
- removed LT-R2: 220, rcl:R-US_0204/7
- removed LT-RC1, LT-RC2: 10uf, resistor:CPOL-EUTT5D9
- removed LT-TRAN: 7805, linear:7805T
- added PCB1, PCB3: ARDUINO_MICRO, E14_Arduino_revB:ARDUINO_MICRO
- CS-ATC1, CS-ATC2, IR-ATC1, IR-ATC2: device capacitor-wima:C2,5-3 -> rcl:C-EU025-024X044
- IR-RC1, IR-RC2: device resistor:CPOL-EUTT5D9 -> resistor:CPOL-EUTT2D5
Connections:
- removed net IRAL: IR-AT.PD5, IR-MULT-LA.A
- removed net IRAR: IR-AT.PD2, IR-MULT-RA.A
- removed net IRBL: IR-AT.PD6, IR-MULT-LA.B
- removed net IRBR: IR-AT.PD3, IR-MULT-RA.B
- removed net IRCL: IR-AT.PD7, IR-MULT-LA.C
- removed net IRCR: IR-AT.PD4, IR-MULT-RA.C
- removed net LTAL: LT-AT.PD5, LT-MULT-1A.A
- removed net LTAR: LT-AT.PD2, LT-MULT-2A.A
- removed net LTBL: LT-AT.PD6, LT-MULT-1A.B
- removed net LTBR: LT-AT.PD3, LT-MULT-2A.B
- removed net LTCL: LT-AT.PD7, LT-MULT-1A.C
- removed net LTCR: LT-AT.PD4, LT-MULT-2A.C
- removed net LTLOUT: LT-AT.PC1, LT-MULT-2A.Y
- removed net LTROUT: LT-AT.PC0, LT-MULT-1A.Y
- removed net LTS1P1: LT-MULT-2A.D1, S1P-6.S
- removed net LTS1P2: LT-MULT-2A.D2, S1P-4.S
- removed net LTS1P3: LT-MULT-2A.D3, S1P-2.S
- removed net LTS2P1: LT-MULT-2A.D4, S2P-6.S
- removed net LTS2P2: LT-MULT-2A.D5, S2P-4.S
- removed net LTS2P3: LT-MULT-2A.D6, S2P-2.S
- removed net LTS3P1: LT-MULT-1A.D1, S3P-6.S
- removed net LTS3P2: LT-MULT-1A.D2, S3P-4.S
- removed net LTS3P3: LT-MULT-1A.D3, S3P-2.S
- removed net LTS4P1: LT-MULT-1A.D4, S4P-6.S
- removed net LTS4P2: LT-MULT-1A.D5, S4P-4.S
- removed net LTS4P3: LT-MULT-1A.D6, S4P-2.S
- removed net N$10: IR-MULT-LA.D1, IRC1L.2, IRR1L.1
- removed net N$12: IR-MULT-RA.D2, IRC2R.1, IRR2R.1
- removed net N$15: IR-MULT-RA.D5, IRC5R.1, IRR5R.2
- removed net N$16: IR-MULT-RA.D6, IRC6R.1, IRR6R.1
- removed net N$17: IR-MULT-RA.D7, IRC7R.2, IRR7R.1
- removed net N$18: IR-MULT-LA.D3, IRC3L.1, IRR3L.1
- removed net N$19: IR-MULT-LA.D4, IRC4L.1, IRR4L.1
- removed net N$22: IR-MULT-LA.D2, IRC2L.1, IRR2L.1
- removed net N$26: IR-MULT-LA.D5, IRC5L.1, IRR5L.2
- removed net N$28: IR-MULT-LA.D6, IRC6L.1, IRR6L.1
- removed net N$3: IR-MULT-RA.D1, IRC1R.2, IRR1R.1
- removed net N$30: IR-MULT-LA.D7, IRC7L.2, IRR7L.1
- removed net N$31: LT-LED.A, LT-R2.1
- removed net N$5: IR-MULT-RA.D3, IRC3R.1, IRR3R.1
- removed net N$6: IR-MULT-RA.D4, IRC4R.1, IRR4R.1
- removed net PB6-A2: LT-AT.PB6, LT-ATC1.2, LT-CR.2
- removed net PB7-A2: LT-AT.PB7, LT-ATC2.2, LT-CR.1
- removed net RESET-AT2: LT-AT.PC6, LT-BTN.A, LT-R1.2
- new net A0: PCB1.A0, S3P-2.S
- new net A0IR: IRC7R.2, IRR7R.1, PCB3.D4
- new net A1: PCB1.A1, S3P-4.S
- new net A10: PCB1.D10, S4P-4.S
- new net A10IR: IRC6L.1, IRR6L.1, PCB3.A4
- new net A11: PCB1.D12, S4P-6.S
- new net A11IR: IRC7L.2, IRR7L.1, PCB3.A5
- new net A1IR: IRC6R.1, IRR6R.1, PCB3.D6
- new net A2: PCB1.A2, S3P-6.S
- new net A2IR: IRC5R.1, IRR5R.2, PCB3.D8
- new net A3: PCB1.A3, S1P-2.S
- new net A3IR: IRC4R.1, IRR4R.1, PCB3.D9
- new net A4: PCB1.A4, S1P-4.S
- new net A4IR: IRC3R.1, IRR3R.1, PCB3.D10
- new net A5: PCB1.A5, S1P-6.S
- new net A5IR: IRC2R.1, IRR2R.1, PCB3.D12
- new net A6: PCB1.D4, S2P-2.S
- new net A6IR: IRC2L.1, IRR2L.1, PCB3.A0
- new net A7: PCB1.D6, S2P-4.S
- new net A7IR: IRC3L.1, IRR3L.1, PCB3.A1
- new net A8: PCB1.D8, S2P-6.S
- new net A8IR: IRC4L.1, IRR4L.1, PCB3.A2
- new net A9: PCB1.D9, S4P-2.S
- new net A9IR: IRC5L.1, IRR5L.2, PCB3.A3
- net +5V-IR: no longer IR-MULT-LP.VCC, IR-MULT-RP.VCC
- net +5V-LT: now also PCB1.+5V; no longer LT-AT.AREF, LT-AT.AVCC, LT-AT.VCC, LT-MULT-1P.VCC, LT-MULT-2P.VCC, LT-R1.1, LT-RC2.+, LT-TRAN.VO, S2P-1.S
- net GND: now also PCB1.GND, PCB1.GND., PCB3.GND, PCB3.GND.; no longer CS-BTN.B, IR-BTN.B, IR-MULT-LA.G, IR-MULT-LP.GND, IR-MULT-RA.G, IR-MULT-RP.GND, LT-AT.GND, LT-AT.GND_2, LT-ATC1.1, LT-ATC2.1, LT-BTN.B, LT-LED.C, LT-MULT-1A.G, LT-MULT-1P.GND, LT-MULT-2A.G, LT-MULT-2P.GND, LT-RC1.+, LT-RC2.-, LT-TRAN.GND
- net IRLOUT: now also IRC1L.2, IRR1L.1; no longer IR-MULT-LA.Y
- net IRROUT: now also IRC1R.2, IRR1R.1; no longer IR-MULT-RA.Y
- net N$32: now also S2P-1.S; no longer LT-AT.PB5, LT-R2.2
- net RESET-AT1: no longer IR-BTN.A
- net RESET-AT3: no longer CS-BTN.A
- net RX-LT: no longer LT-AT.PD0
- net TX-LT: no longer LT-AT.PD1
- net VCC: now also PCB1.VIN, PCB3.VIN; no longer LT-RC1.-, LT-TRAN.VI
Other:
- moved on the sheet: CS-AT, CS-ATC1, CS-ATC2, CS-CR, CS-LED, CS-R1, CS-R2, IR-AT, IR-ATC1, IR-ATC2, IR-CR, IR-LED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

Commit message: ELECTRONICA
FIN DE LOS DISEÑOS
Parts:
- added SV1: (no value), con-lstb:MA05-2
Connections:
- new net +3V3: PCB3.3V3, SV1.7, SV1.8
- new net TX-IR2: IR-AT.PD1, PCB3.RX
- net GND: now also SV1.1, SV1.2; no longer PCB1.GND.
- net RX-IR: no longer IR-AT.PD0
- net RX-LT: now also PCB1.RX
- net SCL: now also PCB3.D3, SV1.5, SV1.6
- net SDA: now also PCB3.D2, SV1.3, SV1.4
- net TX-IR: now also PCB3.TX; no longer IR-AT.PD1
- net TX-LT: now also PCB1.TX
- net VCC: now also SV1.10, SV1.9
Changed lines of the file:
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@@
 <part name="PCB1" library="E14_Arduino_revB" deviceset="ARDUINO_MICRO" device=""/>
 <part name="PCB3" library="E14_Arduino_revB" deviceset="ARDUINO_MICRO" device=""/>
-<part name="GND9" library="supply1" deviceset="GND" device=""/>
-<part name="GND10" library="supply1" deviceset="GND" device=""/>
 <part name="GND11" library="supply1" deviceset="GND" device=""/>
 <part name="GND15" library="supply1" deviceset="GND" device=""/>
@@
 <part name="P+6" library="supply1" deviceset="VCC" device=""/>
 <part name="+5V-LT2" library="supply1" deviceset="+5V" device="" value="+5V-LT"/>
+<part name="SV1" library="con-lstb" deviceset="MA05-2" device=""/>
+<part name="P+1" library="supply1" deviceset="VCC" device=""/>
+<part name="+3V1" library="supply1" deviceset="+3V3" device=""/>
+<part name="+3V2" library="supply1" deviceset="+3V3" device=""/>
+<part name="GND5" library="supply1" deviceset="GND" device=""/>
+<part name="GND8" library="supply1" deviceset="GND" device=""/>
 </parts>
 <sheets>
@@
 <instance part="PCB1" gate="G$1" x="-121.92" y="121.92"/>
 <instance part="PCB3" gate="G$1" x="-50.8" y="121.92"/>
-<instance part="GND9" gate="1" x="-106.68" y="88.9"/>
-<instance part="GND10" gate="1" x="-111.76" y="147.32" rot="R180"/>
 <instance part="GND11" gate="1" x="-40.64" y="149.86" rot="R180"/>
 <instance part="GND15" gate="1" x="-35.56" y="96.52"/>
@@
 <instance part="P+6" gate="VCC" x="-25.4" y="99.06" rot="R270"/>
 <instance part="+5V-LT2" gate="1" x="-111.76" y="96.52" rot="MR180"/>
+<instance part="SV1" gate="G$1" x="0" y="139.7"/>
+<instance part="P+1" gate="VCC" x="15.24" y="149.86"/>
+<instance part="+3V1" gate="G$1" x="-71.12" y="99.06" rot="R90"/>
+<instance part="+3V2" gate="G$1" x="20.32" y="142.24" rot="R270"/>
+<instance part="GND5" gate="1" x="12.7" y="129.54"/>
+<instance part="GND8" gate="1" x="-111.76" y="144.78" rot="R180"/>
 </instances>
 <busses>
@@
 <wire x1="-33.02" y1="104.14" x2="-33.02" y2="99.06" width="0.1524" layer="91"/>
 <wire x1="-33.02" y1="99.06" x2="-27.94" y2="99.06" width="0.1524" layer="91"/>
+</segment>
+<segment>
+<pinref part="SV1" gate="G$1" pin="9"/>
+<pinref part="SV1" gate="G$1" pin="10"/>
+<wire x1="7.62" y1="144.78" x2="-7.62" y2="144.78" width="0.1524" layer="91"/>
+<pinref part="P+1" gate="VCC" pin="VCC"/>
+<wire x1="7.62" y1="144.78" x2="15.24" y2="144.78" width="0.1524" layer="91"/>
+<wire x1="15.24" y1="144.78" x2="15.24" y2="147.32" width="0.1524" layer="91"/>
+<junction x="7.62" y="144.78"/>
 </segment>
 </net>
@@
 </segment>
 <segment>
-<pinref part="PCB1" gate="G$1" pin="GND."/>
-<wire x1="-106.68" y1="104.14" x2="-106.68" y2="91.44" width="0.1524" layer="91"/>
-<pinref part="GND9" gate="1" pin="GND"/>
-</segment>
-<segment>
-<pinref part="PCB1" gate="G$1" pin="GND"/>
-<pinref part="GND10" gate="1" pin="GND"/>
-<wire x1="-111.76" y1="137.16" x2="-111.76" y2="144.78" width="0.1524" layer="91"/>
-</segment>
-<segment>
 <pinref part="GND15" gate="1" pin="GND"/>
 <pinref part="PCB3" gate="G$1" pin="GND."/>
@@
 <wire x1="-40.64" y1="147.32" x2="-40.64" y2="137.16" width="0.1524" layer="91"/>
 </segment>
+<segment>
+<pinref part="SV1" gate="G$1" pin="1"/>
+<pinref part="SV1" gate="G$1" pin="2"/>
+<wire x1="7.62" y1="134.62" x2="-7.62" y2="134.62" width="0.1524" layer="91"/>
+<pinref part="GND5" gate="1" pin="GND"/>
+<wire x1="7.62" y1="134.62" x2="12.7" y2="134.62" width="0.1524" layer="91"/>
+<wire x1="12.7" y1="134.62" x2="12.7" y2="132.08" width="0.1524" layer="91"/>
+<junction x="7.62" y="134.62"/>
+</segment>
+<segment>
+<pinref part="GND8" gate="1" pin="GND"/>
+<pinref part="PCB1" gate="G$1" pin="GND"/>
+<wire x1="-111.76" y1="142.24" x2="-111.76" y2="137.16" width="0.1524" layer="91"/>
+</segment>
 </net>
 <net name="RESET-AT1" class="0">
@@
 <net name="RX-IR" class="0">
 <segment>
-<pinref part="IR-AT" gate="A" pin="PD0"/>
-<wire x1="58.42" y1="43.18" x2="68.58" y2="43.18" width="0.1524" layer="91"/>
-<label x="60.96" y="43.18" size="1.778" layer="95"/>
-</segment>
-<segment>
 <pinref part="TXT" gate="-5" pin="S"/>
 <wire x1="-259.08" y1="96.52" x2="-266.7" y2="96.52" width="0.1524" layer="91"/>
@@
 <net name="TX-IR" class="0">
 <segment>
-<pinref part="IR-AT" gate="A" pin="PD1"/>
-<wire x1="58.42" y1="40.64" x2="68.58" y2="40.64" width="0.1524" layer="91"/>
-<label x="60.96" y="40.64" size="1.778" layer="95"/>
-</segment>
-<segment>
 <pinref part="TXT" gate="-6" pin="S"/>
 <wire x1="-238.76" y1="96.52" x2="-246.38" y2="96.52" width="0.1524" layer="91"/>
 <label x="-246.38" y="96.52" size="1.778" layer="95"/>
+</segment>
+<segment>
+<pinref part="PCB3" gate="G$1" pin="TX"/>
+<wire x1="-33.02" y1="137.16" x2="-33.02" y2="147.32" width="0.1524" layer="91"/>
+<label x="-33.02" y="139.7" size="1.778" layer="95" rot="R90"/>
 </segment>
 </net>
@@
 <label x="-266.7" y="99.06" size="1.778" layer="95"/>
 </segment>
+<segment>
+<pinref part="PCB1" gate="G$1" pin="RX"/>
+<wire x1="-106.68" y1="137.16" x2="-106.68" y2="147.32" width="0.1524" layer="91"/>
+<label x="-106.68" y="139.7" size="1.778" layer="95" rot="R90"/>
+</segment>
 </net>
 <net name="TX-LT" class="0">
@@
 <label x="-246.38" y="99.06" size="1.778" layer="95"/>
 </segment>
+<segment>
+<pinref part="PCB1" gate="G$1" pin="TX"/>
+<wire x1="-104.14" y1="137.16" x2="-104.14" y2="147.32" width="0.1524" layer="91"/>
+<label x="-104.14" y="139.7" size="1.778" layer="95" rot="R90"/>
+</segment>
 </net>
 <net name="+5V-LT" class="0">
@@
 <label x="58.42" y="76.2" size="1.778" layer="95"/>
 </segment>
+<segment>
+<pinref part="SV1" gate="G$1" pin="3"/>
+<wire x1="7.62" y1="137.16" x2="20.32" y2="137.16" width="0.1524" layer="91"/>
+<pinref part="SV1" gate="G$1" pin="4"/>
+<wire x1="7.62" y1="137.16" x2="-7.62" y2="137.16" width="0.1524" layer="91"/>
+<junction x="7.62" y="137.16"/>
+<label x="10.16" y="137.16" size="1.778" layer="95"/>
+</segment>
+<segment>
+<pinref part="PCB3" gate="G$1" pin="D2"/>
+<wire x1="-43.18" y1="137.16" x2="-43.18" y2="147.32" width="0.1524" layer="91"/>
+<label x="-43.18" y="139.7" size="1.778" layer="95" rot="R90"/>
+</segment>
 </net>
 <net name="SCL" class="0">
@@
 <wire x1="55.88" y1="73.66" x2="68.58" y2="73.66" width="0.1524" layer="91"/>
 <label x="58.42" y="73.66" size="1.778" layer="95"/>
+</segment>
+<segment>
+<pinref part="SV1" gate="G$1" pin="5"/>
+<wire x1="7.62" y1="139.7" x2="20.32" y2="139.7" width="0.1524" layer="91"/>
+<pinref part="SV1" gate="G$1" pin="6"/>
+<wire x1="7.62" y1="139.7" x2="-7.62" y2="139.7" width="0.1524" layer="91"/>
+<junction x="7.62" y="139.7"/>
+<label x="10.16" y="139.7" size="1.778" layer="95"/>
+</segment>
+<segment>
+<pinref part="PCB3" gate="G$1" pin="D3"/>
+<wire x1="-45.72" y1="137.16" x2="-45.72" y2="147.32" width="0.1524" layer="91"/>
+<label x="-45.72" y="139.7" size="1.778" layer="95" rot="R90"/>
 </segment>
 </net>
@@
 </segment>
 </net>
+<net name="TX-IR2" class="0">
+<segment>
+<pinref part="IR-AT" gate="A" pin="PD1"/>
+<wire x1="58.42" y1="40.64" x2="68.58" y2="40.64" width="0.1524" layer="91"/>
+<label x="60.96" y="40.64" size="1.778" layer="95"/>
+</segment>
+<segment>
+<pinref part="PCB3" gate="G$1" pin="RX"/>
+<wire x1="-35.56" y1="137.16" x2="-35.56" y2="147.32" width="0.1524" layer="91"/>
+<label x="-35.56" y="139.7" size="1.778" layer="95" rot="R90"/>
+</segment>
+</net>
+<net name="+3V3" class="0">
+<segment>
+<pinref part="+3V1" gate="G$1" pin="+3V3"/>
+<pinref part="PCB3" gate="G$1" pin="3V3"/>
+<wire x1="-68.58" y1="99.06" x2="-66.04" y2="99.06" width="0.1524" layer="91"/>
+<wire x1="-66.04" y1="99.06" x2="-66.04" y2="104.14" width="0.1524" layer="91"/>
+</segment>
+<segment>
+<pinref part="SV1" gate="G$1" pin="7"/>
+<pinref part="SV1" gate="G$1" pin="8"/>
+<wire x1="7.62" y1="142.24" x2="-7.62" y2="142.24" width="0.1524" layer="91"/>
+<pinref part="+3V2" gate="G$1" pin="+3V3"/>
+<wire x1="7.62" y1="142.24" x2="17.78" y2="142.24" width="0.1524" layer="91"/>
+<junction x="7.62" y="142.24"/>
+</segment>
+</net>
