File: electronica/PBC-1/PBC-1.brd (EAGLE design)
At the start: 210 x 199.6 mm, 86 parts

Commit message: diagrama pcb2
diagrama de la pcb de arriba y prueba de la comunicacion serial
Parts:
- IR-TRAN, LT-TRAN: device linear:TO220V -> linear:TO220H
- moved IR-TRAN 12.1 mm to (-51.0, -64.4), turned to 90 degrees
- moved LT-TRAN 9.24 mm to (52.9, 14.3), turned to 315 degrees
- moved IR-RC2 4.43 mm to (47.6, -1.51)
- moved LT-RC2 2.32 mm to (38.2, 1.51)
- moved IR-CR 0.96 mm to (-45.4, 14.6)
Connections:
- net +5V-LT: now also LT-MULT-1.16, LT-MULT-2.16
- net GND: no longer LT-MULT-1.16, LT-MULT-2.16
Routing:
- net GND: track 1059.6 -> 986.0 mm, vias 1 -> 7
- net +5V-LT: track 304.8 -> 337.8 mm, vias 0 -> 1
- net +5V-IR: track 907.7 -> 890.7 mm
- net VCC: track 180.7 -> 196.2 mm
- net IRCR: track 223.5 -> 220.0 mm
- net TX-CS: track 112.6 -> 110.1 mm
- net IRBL: track 54.7 -> 56.6 mm
- net RX-LT: track 74.6 -> 72.9 mm
- net IRCL: track 62.8 -> 61.1 mm
- net IRAR: track 204.7 -> 205.9 mm
- net IRLOUT: track 39.3 -> 38.3 mm
- net LTAR: track 115.4 -> 114.7 mm
- net IRBR: track 212.5 -> 213.2 mm

Commit message: fin pcb-2
fin pcb-2
Parts:
- removed CS-BTN, IR-BTN, LT-BTN: (no value), switch:RDT1034
- removed IR-MULT-L, IR-MULT-R, LT-MULT-1, LT-MULT-2: 74LS151N, 74xx-us:DIL16
- removed LT-AT: ATMEGA328P-PU, Atmel_By_element14_Batch_1-00:DIP254P762X457-28
- removed LT-ATC1, LT-ATC2: 22 pF, capacitor-wima:C2.5-3
- removed LT-CR: 16 MHz, crystal:HC49U70
- removed LT-LED: (no value), led:LED5MM
- removed LT-R1: 10k, rcl:0204/7
- removed LT-R2: 220, rcl:0204/7
- removed LT-RC1, LT-RC2: 10uf, resistor:TT5D9
- removed LT-TRAN: 7805, linear:TO220H
- added PCB1, PCB3: ARDUINO_MICRO, E14_Arduino_revB:ARDUINO_MICRO
- CS-ATC1, CS-ATC2, IR-ATC1, IR-ATC2: device capacitor-wima:C2.5-3 -> rcl:C025-024X044
- IR-RC1, IR-RC2: device resistor:TT5D9 -> resistor:TT2D5
- moved IR-R2 133.2 mm to (60.3, 55.0), turned to 270 degrees
- moved IR-LED 132.8 mm to (55.5, 54.9), turned to 180 degrees
- moved IR-AT 132.2 mm to (70.5, 49.0), turned to 90 degrees
- moved IR-R1 112.1 mm to (65.6, 34.9), turned to 270 degrees
- moved IR-CR 106.1 mm to (58.8, 34.6), turned to 180 degrees
- moved IR-ATC2 102.0 mm to (63.1, 27.8), turned to 180 degrees
- moved IR-ATC1 95.4 mm to (56.2, 27.3), turned to 180 degrees
- moved CS-AT 84.5 mm to (-50.3, -17.4), turned to 180 degrees
- moved TXT 81.7 mm to (-24.8, -80.1), turned to 180 degrees
- moved IR-RC2 77.2 mm to (-22.4, -34.0), turned to 0 degrees
- moved CS-R2 71.6 mm to (-53.7, -31.5), turned to 90 degrees
- moved CS-LED 68.9 mm to (-55.4, -41.1), turned to 0 degrees
- moved CS-ATC2 54.3 mm to (-34.7, -20.9), turned to 180 degrees
- moved IR-TRAN 53.7 mm to (-5.32, -36.2), turned to 270 degrees
- moved CS-CR 46.6 mm to (-36.0, -30.4), turned to 270 degrees
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Connections:
- removed net IRAL: IR-AT.11, IR-MULT-L.11
- removed net IRAR: IR-AT.4, IR-MULT-R.11
- removed net IRBL: IR-AT.12, IR-MULT-L.10
- removed net IRBR: IR-AT.5, IR-MULT-R.10
- removed net IRCL: IR-AT.13, IR-MULT-L.9
- removed net IRCR: IR-AT.6, IR-MULT-R.9
- removed net LTAL: LT-AT.11, LT-MULT-1.11
- removed net LTAR: LT-AT.4, LT-MULT-2.11
- removed net LTBL: LT-AT.12, LT-MULT-1.10
- removed net LTBR: LT-AT.5, LT-MULT-2.10
- removed net LTCL: LT-AT.13, LT-MULT-1.9
- removed net LTCR: LT-AT.6, LT-MULT-2.9
- removed net LTLOUT: LT-AT.24, LT-MULT-2.5
- removed net LTROUT: LT-AT.23, LT-MULT-1.5
- removed net LTS1P1: LT-MULT-2.3, S1P.6
- removed net LTS1P2: LT-MULT-2.2, S1P.4
- removed net LTS1P3: LT-MULT-2.1, S1P.2
- removed net LTS2P1: LT-MULT-2.15, S2P.6
- removed net LTS2P2: LT-MULT-2.14, S2P.4
- removed net LTS2P3: LT-MULT-2.13, S2P.2
- removed net LTS3P1: LT-MULT-1.3, S3P.6
- removed net LTS3P2: LT-MULT-1.2, S3P.4
- removed net LTS3P3: LT-MULT-1.1, S3P.2
- removed net LTS4P1: LT-MULT-1.15, S4P.6
- removed net LTS4P2: LT-MULT-1.14, S4P.4
- removed net LTS4P3: LT-MULT-1.13, S4P.2
- removed net N$10: IR-MULT-L.3, IRC1L.2, IRR1L.1
- removed net N$12: IR-MULT-R.2, IRC2R.1, IRR2R.1
- removed net N$15: IR-MULT-R.14, IRC5R.1, IRR5R.2
- removed net N$16: IR-MULT-R.13, IRC6R.1, IRR6R.1
- removed net N$17: IR-MULT-R.12, IRC7R.2, IRR7R.1
- removed net N$18: IR-MULT-L.1, IRC3L.1, IRR3L.1
- removed net N$19: IR-MULT-L.15, IRC4L.1, IRR4L.1
- removed net N$22: IR-MULT-L.2, IRC2L.1, IRR2L.1
- removed net N$26: IR-MULT-L.14, IRC5L.1, IRR5L.2
- removed net N$28: IR-MULT-L.13, IRC6L.1, IRR6L.1
- removed net N$3: IR-MULT-R.3, IRC1R.2, IRR1R.1
- removed net N$30: IR-MULT-L.12, IRC7L.2, IRR7L.1
- removed net N$31: LT-LED.A, LT-R2.1
- removed net N$5: IR-MULT-R.1, IRC3R.1, IRR3R.1
- removed net N$6: IR-MULT-R.15, IRC4R.1, IRR4R.1
- removed net PB6-A2: LT-AT.9, LT-ATC1.2, LT-CR.2
- removed net PB7-A2: LT-AT.10, LT-ATC2.2, LT-CR.1
- removed net RESET-AT2: LT-AT.1, LT-BTN.A, LT-R1.2
- new net A0: PCB1.A0, S3P.2
- new net A0IR: IRC7R.2, IRR7R.1, PCB3.D4
- new net A1: PCB1.A1, S3P.4
- new net A10: PCB1.D10, S4P.4
- new net A10IR: IRC6L.1, IRR6L.1, PCB3.A4
- new net A11: PCB1.D12, S4P.6
- new net A11IR: IRC7L.2, IRR7L.1, PCB3.A5
- new net A1IR: IRC6R.1, IRR6R.1, PCB3.D6
- new net A2: PCB1.A2, S3P.6
- new net A2IR: IRC5R.1, IRR5R.2, PCB3.D8
- new net A3: PCB1.A3, S1P.2
- new net A3IR: IRC4R.1, IRR4R.1, PCB3.D9
- new net A4: PCB1.A4, S1P.4
- new net A4IR: IRC3R.1, IRR3R.1, PCB3.D10
- new net A5: PCB1.A5, S1P.6
- new net A5IR: IRC2R.1, IRR2R.1, PCB3.D12
- new net A6: PCB1.D4, S2P.2
- new net A6IR: IRC2L.1, IRR2L.1, PCB3.A0
- new net A7: PCB1.D6, S2P.4
- new net A7IR: IRC3L.1, IRR3L.1, PCB3.A1
- new net A8: PCB1.D8, S2P.6
- new net A8IR: IRC4L.1, IRR4L.1, PCB3.A2
- new net A9: PCB1.D9, S4P.2
- new net A9IR: IRC5L.1, IRR5L.2, PCB3.A3
- net +5V-IR: no longer IR-MULT-L.16, IR-MULT-R.16
- net +5V-LT: now also PCB1.+5V; no longer LT-AT.20, LT-AT.21, LT-AT.7, LT-MULT-1.16, LT-MULT-2.16, LT-R1.1, LT-RC2.+, LT-TRAN.3, S2P.1
- net GND: now also PCB1.GND, PCB1.GND., PCB3.GND, PCB3.GND.; no longer CS-BTN.B, IR-BTN.B, IR-MULT-L.7, IR-MULT-L.8, IR-MULT-R.7, IR-MULT-R.8, LT-AT.22, LT-AT.8, LT-ATC1.1, LT-ATC2.1, LT-BTN.B, LT-LED.K, LT-MULT-1.7, LT-MULT-1.8, LT-MULT-2.7, LT-MULT-2.8, LT-RC1.+, LT-RC2.-, LT-TRAN.2
- net IRLOUT: now also IRC1L.2, IRR1L.1; no longer IR-MULT-L.5
- net IRROUT: now also IRC1R.2, IRR1R.1; no longer IR-MULT-R.5
- net N$32: now also S2P.1; no longer LT-AT.19, LT-R2.2
- net RESET-AT1: no longer IR-BTN.A
- net RESET-AT3: no longer CS-BTN.A
- net RX-LT: no longer LT-AT.2
- net TX-LT: no longer LT-AT.3
- net VCC: now also PCB1.VIN, PCB3.VIN; no longer LT-RC1.-, LT-TRAN.1
Routing:
- net GND: track 986.0 -> 0.00 mm, vias 7 -> 0
- net +5V-IR: track 890.7 -> 0.00 mm
- net +5V-LT: track 337.8 -> 0.00 mm, vias 1 -> 0
- net IRCR: track 220.0 -> 0.00 mm
- net IRBR: track 213.2 -> 0.00 mm
- net IRAR: track 205.9 -> 0.00 mm
- net VCC: track 196.2 -> 0.00 mm
- net LTLOUT: track 189.2 -> 0.00 mm
- net IRROUT: track 178.5 -> 0.00 mm
- net TX-LT: track 167.5 -> 0.00 mm
- net N$30: track 134.1 -> 0.00 mm
- net N$17: track 125.1 -> 0.00 mm
- net IRPOUT: track 117.0 -> 0.00 mm
- net LTAR: track 114.7 -> 0.00 mm
- net RX-CS: track 111.4 -> 0.00 mm
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- removed copper zone on layer 1, net GND
- removed copper zone on layer 16, net GND

Commit message: ELECTRONICA
FIN DE LOS DISEÑOS
Parts:
- added SV1: (no value), con-lstb:MA05-2
- moved TXT 30.3 mm to (-27.2, -49.9), turned to 0 degrees
- moved PCB3 5.83 mm to (-70.4, 66.9)
Connections:
- new net +3V3: PCB3.3V3, SV1.7, SV1.8
- new net TX-IR2: IR-AT.3, PCB3.RX1
- net GND: now also SV1.1, SV1.2
- net RX-IR: no longer IR-AT.2
- net RX-LT: now also PCB1.RX1
- net SCL: now also PCB3.D3, SV1.5, SV1.6
- net SDA: now also PCB3.D2, SV1.3, SV1.4
- net TX-IR: now also PCB3.TX1; no longer IR-AT.3
- net TX-LT: now also PCB1.TX1
- net VCC: now also SV1.10, SV1.9
Routing:
- net +5V-IR: track 0.00 -> 964.6 mm
- net A5: track 0.00 -> 507.3 mm
- net A5IR: track 0.00 -> 405.4 mm
- net VCC: track 0.00 -> 365.0 mm
- net A1IR: track 0.00 -> 323.0 mm
- net +5V-LT: track 0.00 -> 236.0 mm, vias 0 -> 1
- net A0IR: track 0.00 -> 215.7 mm
- net A9: track 0.00 -> 215.0 mm
- net A2IR: track 0.00 -> 187.1 mm
- net A3IR: track 0.00 -> 181.9 mm
- net A11IR: track 0.00 -> 159.8 mm
- net A4IR: track 0.00 -> 157.3 mm
- net A7: track 0.00 -> 142.6 mm
- net TX-IR: track 0.00 -> 139.4 mm
- net A3: track 0.00 -> 136.2 mm, vias 0 -> 4
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- added copper zone on layer 1, net GND
- added copper zone on layer 16, net GND
Other:
- board text added: "C:/Users/carlos hugo/Desktop/github/L16/electronica/PBC-2/InteliRobot.bmp"

Commit message: ELECTRONICA FIN
diseño final de las pcb's y creacion de gerbers
Routing:
- net +5V-IR: track 964.6 -> 959.9 mm
- net TX-IR: track 139.4 -> 142.2 mm
- net A1IR: track 323.0 -> 324.4 mm
- net A5: track 507.3 -> 508.6 mm
- net A4: track 129.1 -> 130.2 mm
- net VCC: track 365.0 -> 364.4 mm
- net N$2: track 2.85 -> 2.29 mm
